Commit message: visualizing IK solutions; smart pointers instead of raw pointers; updated module tests

File: RobotSystems/Valkyrie/valkyrie_simple.urdf (robot description, URDF)
Before this commit: robot valkyrie, 76 links, 75 joints
Links:
- link head: geometry collision box size=0.0468 0.12 0.1184; collision box size=0.1311 0.12 0.0591
- link hokuyo_link: geometry collision box size=0.08 0.06 0.04238; collision cylinder length=0.047 radius=0.024425
- link leftAnklePitchLink: geometry collision mesh filename=package://val_dynacore/RobotSystems/Valkyrie/model/meshes/l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; visual mesh filename=package://val_dynacore/RobotSystems/Valkyrie/model/meshes/l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
- link leftElbowPitchLink: geometry collision mesh filename=package://val_dynacore/RobotSystems/Valkyrie/model/meshes/a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; visual mesh filename=package://val_dynacore/RobotSystems/Valkyrie/model/meshes/a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
- link leftFoot: geometry collision box size=0.27 0.16 0.064; visual mesh filename=package://val_dynacore/RobotSystems/Valkyrie/model/meshes/l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
- link leftForearmLink: geometry collision mesh filename=package://val_dynacore/RobotSystems/Valkyrie/model/meshes/a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; visual mesh filename=package://val_dynacore/RobotSystems/Valkyrie/model/meshes/a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
- link leftHipPitchLink: geometry collision mesh filename=package://val_dynacore/RobotSystems/Valkyrie/model/meshes/l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; visual mesh filename=package://val_dynacore/RobotSystems/Valkyrie/model/meshes/l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
- link leftHipRollLink: geometry collision mesh filename=package://val_dynacore/RobotSystems/Valkyrie/model/meshes/l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; visual mesh filename=package://val_dynacore/RobotSystems/Valkyrie/model/meshes/l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
- link leftHipYawLink: geometry collision mesh filename=package://val_dynacore/RobotSystems/Valkyrie/model/meshes/l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; visual mesh filename=package://val_dynacore/RobotSystems/Valkyrie/model/meshes/l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
- link leftIndexFingerPitch1Link: geometry collision mesh filename=package://val_dynacore/RobotSystems/Valkyrie/model/meshes/f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; visual mesh filename=package://val_dynacore/RobotSystems/Valkyrie/model/meshes/f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
- link leftIndexFingerPitch2Link: geometry collision mesh filename=package://val_dynacore/RobotSystems/Valkyrie/model/meshes/f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; visual mesh filename=package://val_dynacore/RobotSystems/Valkyrie/model/meshes/f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
- link leftIndexFingerPitch3Link: geometry collision mesh filename=package://val_dynacore/RobotSystems/Valkyrie/model/meshes/f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; visual mesh filename=package://val_dynacore/RobotSystems/Valkyrie/model/meshes/f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
- link leftKneePitchLink: geometry collision mesh filename=package://val_dynacore/RobotSystems/Valkyrie/model/meshes/l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; visual mesh filename=package://val_dynacore/RobotSystems/Valkyrie/model/meshes/l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
- link leftMiddleFingerPitch1Link: geometry collision mesh filename=package://val_dynacore/RobotSystems/Valkyrie/model/meshes/f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; visual mesh filename=package://val_dynacore/RobotSystems/Valkyrie/model/meshes/f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
- link leftMiddleFingerPitch2Link: geometry collision mesh filename=package://val_dynacore/RobotSystems/Valkyrie/model/meshes/f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; visual mesh filename=package://val_dynacore/RobotSystems/Valkyrie/model/meshes/f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
- link leftMiddleFingerPitch3Link: geometry collision mesh filename=package://val_dynacore/RobotSystems/Valkyrie/model/meshes/f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; visual mesh filename=package://val_dynacore/RobotSystems/Valkyrie/model/meshes/f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
- link leftPalm: geometry collision mesh filename=package://val_dynacore/RobotSystems/Valkyrie/model/meshes/a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; visual mesh filename=package://val_dynacore/RobotSystems/Valkyrie/model/meshes/a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
- link leftPinkyPitch1Link: geometry collision mesh filename=package://val_dynacore/RobotSystems/Valkyrie/model/meshes/f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; visual mesh filename=package://val_dynacore/RobotSystems/Valkyrie/model/meshes/f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
- link leftPinkyPitch2Link: geometry collision mesh filename=package://val_dynacore/RobotSystems/Valkyrie/model/meshes/f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; visual mesh filename=package://val_dynacore/RobotSystems/Valkyrie/model/meshes/f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
- link leftPinkyPitch3Link: geometry collision mesh filename=package://val_dynacore/RobotSystems/Valkyrie/model/meshes/f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; visual mesh filename=package://val_dynacore/RobotSystems/Valkyrie/model/meshes/f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
- link leftShoulderPitchLink: geometry collision mesh filename=package://val_dynacore/RobotSystems/Valkyrie/model/meshes/a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; visual mesh filename=package://val_dynacore/RobotSystems/Valkyrie/model/meshes/a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
- link leftShoulderRollLink: geometry collision mesh filename=package://val_dynacore/RobotSystems/Valkyrie/model/meshes/a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; visual mesh filename=package://val_dynacore/RobotSystems/Valkyrie/model/meshes/a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
- link leftShoulderYawLink: geometry collision mesh filename=package://val_dynacore/RobotSystems/Valkyrie/model/meshes/a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; visual mesh filename=package://val_dynacore/RobotSystems/Valkyrie/model/meshes/a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
- link leftThumbPitch1Link: geometry collision mesh filename=package://val_dynacore/RobotSystems/Valkyrie/model/meshes/f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; visual mesh filename=package://val_dynacore/RobotSystems/Valkyrie/model/meshes/f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
- link leftThumbPitch2Link: geometry collision mesh filename=package://val_dynacore/RobotSystems/Valkyrie/model/meshes/f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; visual mesh filename=package://val_dynacore/RobotSystems/Valkyrie/model/meshes/f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
- link leftThumbPitch3Link: geometry collision mesh filename=package://val_dynacore/RobotSystems/Valkyrie/model/meshes/f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; visual mesh filename=package://val_dynacore/RobotSystems/Valkyrie/model/meshes/f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
- link leftThumbRollLink: geometry collision mesh filename=package://val_dynacore/RobotSystems/Valkyrie/model/meshes/f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; visual mesh filename=package://val_dynacore/RobotSystems/Valkyrie/model/meshes/f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
- link leftWristRollLink: geometry collision mesh filename=package://val_dynacore/RobotSystems/Valkyrie/model/meshes/a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; visual mesh filename=package://val_dynacore/RobotSystems/Valkyrie/model/meshes/a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
- link lowerNeckPitchLink: geometry collision mesh filename=package://val_dynacore/RobotSystems/Valkyrie/model/meshes/h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; visual mesh filename=package://val_dynacore/RobotSystems/Valkyrie/model/meshes/h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
- link neckYawLink: geometry collision mesh filename=package://val_dynacore/RobotSystems/Valkyrie/model/meshes/h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; visual mesh filename=package://val_dynacore/RobotSystems/Valkyrie/model/meshes/h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
- link pelvis: geometry collision mesh filename=package://val_dynacore/RobotSystems/Valkyrie/model/meshes/p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; visual mesh filename=package://val_dynacore/RobotSystems/Valkyrie/model/meshes/p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
- link rightAnklePitchLink: geometry collision mesh filename=package://val_dynacore/RobotSystems/Valkyrie/model/meshes/l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; visual mesh filename=package://val_dynacore/RobotSystems/Valkyrie/model/meshes/l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
- link rightElbowPitchLink: geometry collision mesh filename=package://val_dynacore/RobotSystems/Valkyrie/model/meshes/a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; visual mesh filename=package://val_dynacore/RobotSystems/Valkyrie/model/meshes/a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
- link rightFoot: geometry collision box size=0.27 0.16 0.064; visual mesh filename=package://val_dynacore/RobotSystems/Valkyrie/model/meshes/l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
- link rightForearmLink: geometry collision mesh filename=package://val_dynacore/RobotSystems/Valkyrie/model/meshes/a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; visual mesh filename=package://val_dynacore/RobotSystems/Valkyrie/model/meshes/a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
- link rightHipPitchLink: geometry collision mesh filename=package://val_dynacore/RobotSystems/Valkyrie/model/meshes/l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; visual mesh filename=package://val_dynacore/RobotSystems/Valkyrie/model/meshes/l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
- link rightHipRollLink: geometry collision mesh filename=package://val_dynacore/RobotSystems/Valkyrie/model/meshes/l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; visual mesh filename=package://val_dynacore/RobotSystems/Valkyrie/model/meshes/l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
- link rightHipYawLink: geometry collision mesh filename=package://val_dynacore/RobotSystems/Valkyrie/model/meshes/l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; visual mesh filename=package://val_dynacore/RobotSystems/Valkyrie/model/meshes/l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
- link rightIndexFingerPitch1Link: geometry collision mesh filename=package://val_dynacore/RobotSystems/Valkyrie/model/meshes/f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; visual mesh filename=package://val_dynacore/RobotSystems/Valkyrie/model/meshes/f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
- link rightIndexFingerPitch2Link: geometry collision mesh filename=package://val_dynacore/RobotSystems/Valkyrie/model/meshes/f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; visual mesh filename=package://val_dynacore/RobotSystems/Valkyrie/model/meshes/f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
- link rightIndexFingerPitch3Link: geometry collision mesh filename=package://val_dynacore/RobotSystems/Valkyrie/model/meshes/f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; visual mesh filename=package://val_dynacore/RobotSystems/Valkyrie/model/meshes/f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
- link rightKneePitchLink: geometry collision mesh filename=package://val_dynacore/RobotSystems/Valkyrie/model/meshes/l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; visual mesh filename=package://val_dynacore/RobotSystems/Valkyrie/model/meshes/l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
- link rightMiddleFingerPitch1Link: geometry collision mesh filename=package://val_dynacore/RobotSystems/Valkyrie/model/meshes/f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; visual mesh filename=package://val_dynacore/RobotSystems/Valkyrie/model/meshes/f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
- link rightMiddleFingerPitch2Link: geometry collision mesh filename=package://val_dynacore/RobotSystems/Valkyrie/model/meshes/f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; visual mesh filename=package://val_dynacore/RobotSystems/Valkyrie/model/meshes/f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
- link rightMiddleFingerPitch3Link: geometry collision mesh filename=package://val_dynacore/RobotSystems/Valkyrie/model/meshes/f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; visual mesh filename=package://val_dynacore/RobotSystems/Valkyrie/model/meshes/f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
- link rightPalm: geometry collision mesh filename=package://val_dynacore/RobotSystems/Valkyrie/model/meshes/a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; visual mesh filename=package://val_dynacore/RobotSystems/Valkyrie/model/meshes/a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
- link rightPinkyPitch1Link: geometry collision mesh filename=package://val_dynacore/RobotSystems/Valkyrie/model/meshes/f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; visual mesh filename=package://val_dynacore/RobotSystems/Valkyrie/model/meshes/f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
- link rightPinkyPitch2Link: geometry collision mesh filename=package://val_dynacore/RobotSystems/Valkyrie/model/meshes/f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; visual mesh filename=package://val_dynacore/RobotSystems/Valkyrie/model/meshes/f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
- link rightPinkyPitch3Link: geometry collision mesh filename=package://val_dynacore/RobotSystems/Valkyrie/model/meshes/f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; visual mesh filename=package://val_dynacore/RobotSystems/Valkyrie/model/meshes/f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
- link rightShoulderPitchLink: geometry collision mesh filename=package://val_dynacore/RobotSystems/Valkyrie/model/meshes/a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; visual mesh filename=package://val_dynacore/RobotSystems/Valkyrie/model/meshes/a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
- link rightShoulderRollLink: geometry collision mesh filename=package://val_dynacore/RobotSystems/Valkyrie/model/meshes/a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; visual mesh filename=package://val_dynacore/RobotSystems/Valkyrie/model/meshes/a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
- link rightShoulderYawLink: geometry collision mesh filename=package://val_dynacore/RobotSystems/Valkyrie/model/meshes/a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; visual mesh filename=package://val_dynacore/RobotSystems/Valkyrie/model/meshes/a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
- link rightThumbPitch1Link: geometry collision mesh filename=package://val_dynacore/RobotSystems/Valkyrie/model/meshes/f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; visual mesh filename=package://val_dynacore/RobotSystems/Valkyrie/model/meshes/f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
- link rightThumbPitch2Link: geometry collision mesh filename=package://val_dynacore/RobotSystems/Valkyrie/model/meshes/f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; visual mesh filename=package://val_dynacore/RobotSystems/Valkyrie/model/meshes/f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
- link rightThumbPitch3Link: geometry collision mesh filename=package://val_dynacore/RobotSystems/Valkyrie/model/meshes/f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; visual mesh filename=package://val_dynacore/RobotSystems/Valkyrie/model/meshes/f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
- link rightThumbRollLink: geometry collision mesh filename=package://val_dynacore/RobotSystems/Valkyrie/model/meshes/f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; visual mesh filename=package://val_dynacore/RobotSystems/Valkyrie/model/meshes/f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
- link rightWristRollLink: geometry collision mesh filename=package://val_dynacore/RobotSystems/Valkyrie/model/meshes/a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; visual mesh filename=package://val_dynacore/RobotSystems/Valkyrie/model/meshes/a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
- link torso: geometry collision mesh filename=package://val_dynacore/RobotSystems/Valkyrie/model/meshes/t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; visual mesh filename=package://val_dynacore/RobotSystems/Valkyrie/model/meshes/t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
- link torsoPitchLink: geometry collision mesh filename=package://val_dynacore/RobotSystems/Valkyrie/model/meshes/t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; visual mesh filename=package://val_dynacore/RobotSystems/Valkyrie/model/meshes/t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
- link torsoYawLink: geometry collision mesh filename=package://val_dynacore/RobotSystems/Valkyrie/model/meshes/t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; visual mesh filename=package://val_dynacore/RobotSystems/Valkyrie/model/meshes/t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
- link upperNeckPitchLink: geometry collision mesh filename=package://val_dynacore/RobotSystems/Valkyrie/model/meshes/h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; visual mesh filename=package://val_dynacore/RobotSystems/Valkyrie/model/meshes/h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
